File: hardware/Battery_Monitor.kicad_sch (KiCad schematic)
At the start: 6 parts, among them U301 STC3100IQT

Commit message: Add battery protection and swap some connectors
Parts:
- R302: value 0.01 -> 0.03
Changed lines of the file:
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@@
 	(title_block
 		(title "BT Bike Light")
-		(date "2024-08-24")
+		(date "2024-08-25")
 		(rev "A")
 		(company "Embedded Shark, LLC")
@@
 			)
 		)
-		(property "Value" "0.01"
+		(property "Value" "0.03"
 			(at 154.432 102.87 0)
 			(effects
