File: hardware/LED_Driver.kicad_sch (KiCad schematic)
At the start: 5 parts, among them U501 PAM2808

Commit message: Add battery protection and swap some connectors
Connections:
- net +BATT: now reaches C501.1, U501.2 (VIN)
Changed lines of the file:
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@@
 	(title_block
 		(title "BT Bike Light")
-		(date "2024-08-24")
+		(date "2024-08-25")
 		(rev "A")
 		(company "Embedded Shark, LLC")
@@
 		(color 0 0 0 0)
 	)
+	(junction
+		(at 118.11 87.63)
+		(diameter 0)
+		(color 0 0 0 0)
+	)
 	(no_connect
 		(at 167.64 92.71)
@@
 		(pts
 			(xy 153.67 97.79) (xy 153.67 90.17)
+		)
+		(stroke
+			(width 0)
+			(type default)
+		)
+	)
+	(wire
+		(pts
+			(xy 118.11 86.36) (xy 118.11 87.63)
 		)
 		(stroke
@@
 		(dnp no)
 		(fields_autoplaced yes)
-		(property "Reference" "#PWR0501"
+		(property "Reference" "#PWR0502"
 			(at 118.11 111.76 0)
 			(effects
@@
 		(instances
 			(project "BT-Bike-Light"
+				(path "/3263b444-391f-435a-aeab-6f7fca8830e2/ec5dace2-0a24-46f6-a2b0-71991eb2cd39"
+					(reference "#PWR0502")
+					(unit 1)
+				)
+			)
+		)
+	)
+	(symbol
+		(lib_id "power:+BATT")
+		(at 118.11 86.36 0)
+		(unit 1)
+		(exclude_from_sim no)
+		(in_bom yes)
+		(on_board yes)
+		(dnp no)
+		(fields_autoplaced yes)
+		(property "Reference" "#PWR0501"
+			(at 118.11 90.17 0)
+			(effects
+				(font
+					(size 1.27 1.27)
+				)
+				(hide yes)
+			)
+		)
+		(property "Value" "+BATT"
+			(at 118.11 81.28 0)
+			(effects
+				(font
+					(size 1.27 1.27)
+				)
+			)
+		)
+		(property "Footprint" ""
+			(at 118.11 86.36 0)
+			(effects
+				(font
+					(size 1.27 1.27)
+				)
+				(hide yes)
+			)
+		)
+		(property "Datasheet" ""
+			(at 118.11 86.36 0)
+			(effects
+				(font
+					(size 1.27 1.27)
+				)
+				(hide yes)
+			)
+		)
+		(property "Description" "Power symbol creates a global label with name \"+BATT\""
+			(at 118.11 86.36 0)
+			(effects
+				(font
+					(size 1.27 1.27)
+				)
+				(hide yes)
+			)
+		)
+		(pin "1"
+		)
+		(instances
+			(project ""
 				(path "/3263b444-391f-435a-aeab-6f7fca8830e2/ec5dace2-0a24-46f6-a2b0-71991eb2cd39"
 					(reference "#PWR0501")
@@
 		(dnp no)
 		(fields_autoplaced yes)
-		(property "Reference" "#PWR0503"
+		(property "Reference" "#PWR0504"
 			(at 162.56 111.76 0)
 			(effects
@@
 			(project "BT-Bike-Light"
 				(path "/3263b444-391f-435a-aeab-6f7fca8830e2/ec5dace2-0a24-46f6-a2b0-71991eb2cd39"
-					(reference "#PWR0503")
+					(reference "#PWR0504")
 					(unit 1)
 				)
@@
 		(dnp no)
 		(fields_autoplaced yes)
-		(property "Reference" "#PWR0502"
+		(property "Reference" "#PWR0503"
 			(at 132.08 111.76 0)
 			(effects
@@
 			(project "BT-Bike-Light"
 				(path "/3263b444-391f-435a-aeab-6f7fca8830e2/ec5dace2-0a24-46f6-a2b0-71991eb2cd39"
-					(reference "#PWR0502")
+					(reference "#PWR0503")
 					(unit 1)
 				)
@@
 		(dnp no)
 		(fields_autoplaced yes)
-		(property "Reference" "#PWR0504"
+		(property "Reference" "#PWR0505"
 			(at 172.72 111.76 0)
 			(effects
@@
 			(project "BT-Bike-Light"
 				(path "/3263b444-391f-435a-aeab-6f7fca8830e2/ec5dace2-0a24-46f6-a2b0-71991eb2cd39"
-					(reference "#PWR0504")
-					(unit 1)
-				)
+					(reference "#PWR0505")
+					(unit 1)
+				)
